File: Solar analyzer/Measuringmeter/OneSchematicToRuleThemAll.sch (EAGLE design)
At the start: 162 parts, among them J1 105133-0001, J2 105133-0001, U1 ATMEGA328P-AU, U2 Value, U3 MAX13253ATB+T21-0137I_T1033-1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, X1 TRANSFORMER, X2 TRANSFORMER

Commit message: add discharge Resister and Relay
Parts:
- added R38, R39: 100M, VoltagemeasurementComponents:HVA12FA100M
- added R40: (no value), Ampparts:RX0402_100
- added RDIS1: 200M, CAP_Diode_Megger:RESISTOR20OHM
- added U$39: (no value), CAP_Diode_Megger:REEDRELAYSPDT
- R15, R16, R17, R18, R19, R20: value (none) -> 100M; device VoltagemeasurementComponents:HVA05FA100M -> VoltagemeasurementComponents:HVA12FA100M
- R21, R22, R23, R24: value (none) -> 348k
- U$29: value RESISTOR200MOHM -> SI2302A; device CAP_Diode_Megger:RESISTOR20OHM -> Ampparts:SI2302A; SPICEPREFIX R -> (none)
Connections:
- new net DISCHARGE: R40.1, U$21.Y5
- new net N$90: R38.2, R39.1
- new net N$91: U$29.D, U$39.2
- new net N$92: R40.2, U$29.G
- new net N$93: RDIS1.2, U$39.1
- net +5V: now also U$39.3
- net GND: now also U$29.S
- net HV-: now also RDIS1.1
- net MEG-: now also R39.2; no longer U$29.2
- net N$50: now also R38.1; no longer U$29.1
- net N$57: now also PTC2.P$2, R20.2; no longer R15.1
- net N$58: now also R15.2, R16.1; no longer R17.1, R19.2
- net N$59: now also R15.1, R18.1; no longer R19.1, R20.1
- net N$61: now also R16.2, R17.1; no longer R16.1, R18.2
- net N$62: now also R18.2, R19.1; no longer R18.1, R20.2
- net N$65: now also R19.2, R20.1; no longer PTC2.P$2, R15.2, R16.2
- net VOUT5000: now also U$39.4
Other:
- note added: "Isolate the frick out of this HV- GND"
- note added: "Place RS1 close to Amplifier and ground plane Reduce the trace lenth to the path"
- note removed: "Place RS1 close Amplifier and ground plane Reduce the trace lenth to the path"
- moved on the sheet: ADC1, ADC2, C1, C10, C11, C12, C13, C14, C2, C3, C4, C5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

Commit message: Add instrumentation amplifiers
Parts:
- removed C11: (no value), powersupply:EMK107B7105KA-T
- removed U$25: (no value), CAP_Diode_Megger:CAPACTORFORTRANSFORMER
- removed U$29, U$32, U$34, U$35, U$36, U$37, U$38: SI2302A, Ampparts:SI2302A
- removed U$30, U$31: (no value), Ampparts:OPA300-ND
- added ADC3: ADS1115IDGSR, Ampparts:ADS1115IDGSR
- added C15: 1uF, powersupply:EMK107B7105KA-T
- added C16: 1uf, powersupply:EMK107B7105KA-T
- added C17: 1e-7, powersupply:CC0402KRX5R7BB104
- added C18: (no value), powersupply:CC0402KRX5R7BB104
- added FB10, FB5, FB6, FB9: (no value), Ampparts:MMZ2012Y152BT000
- added IC1, IC2: (no value), Ampparts:INA333
- added J3: 22-05-7028-02, con-molex:22-05-7028-02
- added R41, R42, R43, R44: 10k, Ampparts:ERJ-3GEYJ103V
- added R45, R47, R53: (no value), Ampparts:RX0402_100
- added R48, R49, R50, R51: 10K, Ampparts:ERJ-2GEJ102X
- added R52, R54: (no value), Ampparts:ERJ-3GEYJ103V
- added S2: (no value), switch-omron:31-XX
- added S3: Voltage Measurement, switch-omron:31-XX
- added S4: Current measurement, switch-omron:31-XX
- added S5: megger ON, switch-omron:31-XX
- added S6: voltage selection 1, switch-omron:31-XX
- added S7: ENTER, switch-omron:31-XX
- added S8: EMERGENCY STOP, switch-omron:31-XX
- added T1, T10, T2, T3, T4, T5, T6, T8, U$44: SI2302A, Ampparts:SI2302A
- added T11, T9: (no value), Ampparts:NX2301P,215
- R8: value (none) -> 10K
- SMD1: SPICEPREFIX C -> (none)
- U$24: value (none) -> 15uF
- U$26: value SI2302A -> 100nF; device Ampparts:SI2302A -> powersupply:CC0402KRX5R7BB104
- U$27: value (none) -> 100nF; device Ampparts:RX0402_100 -> powersupply:CC0402KRX5R7BB104
Connections:
- removed net N$92: R40.2, U$29.G
- removed net TO5+: J1.VBUS, J2.VBUS, JP1.2, JP2.1, U$25.P$2, U1.AREF, U1.AVCC, U1.VCC
- removed net TOADC: ADC2.AIN0, ADC2.AIN1, ADC2.AIN2, ADC2.AIN3, U$31.IN-, U$31.OUT
- removed net TOBAT-: S1.S
- removed net TOMCFORFAULTDETECTION: U3.!FAULT
- new net FAULTMAXIC: R48.2, U$19.GPIO18
- new net N$100: ADC3.VDD, C15.2, C16.1, FB6.P$1, R41.2, R42.2, R43.2
- new net N$101: ADC3.AIN1, ADC3.AIN3, J3-1.S
- new net N$102: R45.2, U$44.G
- new net N$103: FB5.P$1, U$44.D
- new net N$105: FB9.P$2, T8.S
- new net N$106: S3.S, U$19.GPIO4/GCKL
- new net N$107: S4.S, U$19.GPIO17/GEN0
- new net N$108: S5.S, U$19.GPIO27/GEN2
- new net N$109: S6.S, U$19.GPIO22/GEN3
- new net N$110: S7.S, U$19.GPIO10/MOSI
- new net N$111: R50.2, S3.P, S4.P, S5.P, S6.P, S7.P
- new net N$112: S8.P, U$19.GEN/6GPIO25
- new net N$113: R51.2, S8.S
- new net N$114: FB2.P$1, T9.S
- new net N$115: R54.1, T10.D, T11.G
- new net N$116: ADC1.VDD, C10.1, C17.1, C9.2, IC1.+VS, R25.2, R26.2, R27.2, T9.D
- new net N$117: C12.2, C13.1, C18.2, IC2.+VS, T11.D
- new net N$118: ADC1.AIN0, ADC1.AIN2, IC1.OUT
- new net N$119: ADC2.AIN0, ADC2.AIN2, IC2.OUT
- new net N$94: ADC3.ADDR, R44.2
- new net N$95: ADC3.SCL, R41.1, R44.1
- new net N$96: ADC3.SDA, R42.1
- new net N$97: ADC3.AIN0, ADC3.AIN2, J3-2.S
- new net N$98: ADC3.ALERT/RDY, R43.1
- new net N$99: ADC3.GND, C15.1, C16.2, FB5.P$2
- new net TOATMEGAVCC: C6.1, C7.1, JP1.2, JP2.1, L1.P$2, R49.1, U$18.SYS, U$26.2, U1.AVCC, U1.VCC
- net +5V: now also FB10.P$1, FB6.P$2, R52.2, R54.2, U$20.VCC, U$21.VCC, U$22.VCC, U$23.VCC, U$24.P$1; no longer C11.2, U$30.V+
- net GND: now also ADC1.AIN1, ADC1.AIN3, ADC2.AIN1, ADC2.AIN3, C17.2, C18.1, FB1.P$1, FB3.P$1, FB9.P$1, IC1.-IN, IC1.-VS, IC1.REF, IC2.-IN, IC2.-VS, IC2.REF, J2.SHIELD, R28.1, R50.1, R51.1, S1.S, S2.S, T1.S, T10.S, T2.S, T3.S, T4.S, T5.S, T6.S, T8.D, U$26.1, U$27.2, U$44.S; no longer U$25.P$1, U$26.D, U$26.S, U$29.S, U$32.S, U$34.S, U$35.S, U$36.S, U$37.S, U$38.S
- net N$16: now also R53.2; no longer C11.1, FB1.P$1, R28.1, U$30.V-, U$38.D
- net N$2: now also U$27.1, U1.AREF; no longer C6.1, C7.1, L1.P$2, U$18.SYS
- net N$27: now also R48.1, U3.!FAULT; no longer U$20.VCC, U$21.VCC, U$22.VCC, U$23.VCC, U$24.P$1
- net N$29: now also R47.2, T8.G; no longer U$26.G, U$27.1
- net N$50: now also IC2.+IN; no longer U$31.IN+
- net N$51: now also FB10.P$2, J1.VBUS, J2.VBUS; no longer FB3.P$1, U$31.V-, U$32.D
- net N$53: now also T2.D, U$39.2; no longer U$34.D, U$43.2
- net N$54: now also R40.2, T2.G; no longer U$35.D, U$42.2
- net N$55: now also R34.2, T3.G; no longer U$36.D, U$41.2
- net N$56: now also T3.D, U$43.2; no longer U$37.D, U$40.2
- net N$59: now also IC1.+IN; no longer U$30.IN+
- net N$64: now also FB4.P$1, T11.S; no longer ADC1.AIN0, ADC1.AIN1, ADC1.AIN2, ADC1.AIN3, U$30.IN-, U$30.OUT
- net N$76: now also R52.1, T1.D, T9.G; no longer ADC1.VDD, C10.1, C9.2, FB2.P$1, R25.2, R26.2, R27.2
- net N$79: no longer U$38.G
- net N$80: now also R35.1, T4.G; no longer R34.2, U$34.G
- net N$86: no longer C12.2, C13.1, FB4.P$1, U$31.V+
- net N$87: now also R36.1, T5.G; no longer R35.1, U$35.G
- net N$88: now also T5.D, U$41.2; no longer R36.1, U$36.G
- net N$89: now also T6.G; no longer U$37.G
- net N$91: now also T6.D, U$40.2; no longer U$29.D, U$39.2
- net PRM2: no longer U$32.G
- net PRM3: now also R45.1
- net RESET: now also R49.2, S2.P
- net SWITCHON: now also R47.1; no longer U$27.2
Other:
- note added: "ADD BANANA CONNECTOR"
- note added: "Connectors to power Pi and the display. easier to drill a hole in the middle of the PCB for ease of attaching the microUSB cable (MicroUSB turnt out to be the only way of of powering the pi reliably)"
- note added: "Second capacitor near the supply orgin"
- note removed: "Connectors to power Pi and the display neer to drill a hole in the middle of the PCB for ease of attaching the microUSB cable (MicroUSB turnt out to be the only way of of powering the pi reliably)"
- moved on the sheet: ADC1, C1, C10, C2, C3, C4, C5, C6, C7, C8, C9, D1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

Commit message: Add relays
In voltage measurement and to select the voltage in megger. Add p-channel mosfet to power pi and decoder
Parts:
- removed FB10, FB9: (no value), Ampparts:MMZ2012Y152BT000
- removed R35: (no value), Ampparts:RX0402_100
- removed T4: SI2302A, Ampparts:SI2302A
- removed U$40, U$41, U$42, U$43: (no value), CAP_Diode_Megger:REEDRELAYSPDT
- added C11: (no value), powersupply:CC0402KRX5R7BB104
- added C19: 1e-7, powersupply:CC0402KRX5R7BB104
- added JP3: (no value), jumper:JP1E
- added JP4: (no value), jumper:JP2E
- added R46: 10k, Ampparts:ERJ-3GEYJ103V
- added R55, R56, R57, R58, R59, R60: (no value), Ampparts:RX0402_100
- added REEDRELAY1, REEDRELAY2, REEDRELAY3, REEDRELAY4: (no value), CAP_Diode_Megger:REEDRELAYSPDT
- added RELAY1, RELAY2, RELAY3, RELAY4, RELAY5: (no value), CAP_Diode_Megger:T9GS1L14-5
- added T12, T13, T14, T15, T16, T17: SI2302A, Ampparts:SI2302A
- added T7: (no value), Ampparts:NX2301P,215
- added U$25, U$29: (no value), Ampparts:OPA300-ND
- R34: value (none) -> 10k; device Ampparts:RX0402_100 -> Ampparts:ERJ-3GEYJ103V
- T3: value SI2302A -> (none); device Ampparts:SI2302A -> Ampparts:NX2301P,215
Connections:
- removed net MEG+: U$40.1, U$41.1, U$42.1, U$43.1
- removed net N$105: FB9.P$2, T8.S
- removed net N$51: FB10.P$2, J1.VBUS, J2.VBUS
- removed net N$87: R36.1, T5.G
- removed net N$88: T5.D, U$41.2
- removed net VOUT5000: SMD38.P$2, SMD40.C, U$39.4, U$40.4
- new net N$104: IC2.OUT, U$29.IN+
- new net N$120: C11.1, C12.2, C13.1, C18.2, IC2.+VS, T11.D, U$29.V+
- new net N$121: ADC1.GND, FB1.P$2
- new net N$122: R36.2, T5.G
- new net N$125: RELAY2.C2, T14.D
- new net N$126: RELAY3.C2, T13.D
- new net N$127: RELAY4.C2, T12.D
- new net N$128: RELAY1.C2, T15.D
- new net N$129: R55.2, T15.G
- new net N$130: R56.1, T14.G
- new net N$131: R57.1, T13.G
- new net N$132: R58.2, T12.G
- new net N$133: R60.2, T6.G
- new net N$134: REEDRELAY2.3, T6.D
- new net N$136: REEDRELAY3.3, T17.D
- new net N$137: R59.1, T17.G
- new net N$92: R37.1, T16.G
- new net PIE5+: J1.VBUS, J2.VBUS, T3.D, U$20.VCC, U$21.VCC, U$22.VCC, U$23.VCC, U$24.P$1
- new net POWERON: U1.PD7, U2.EN
- new net VOUTHV: JP3.2, SMD38.P$2, SMD40.C, U$39.4
- net +5V: now also R34.2, R46.2, REEDRELAY1.2, REEDRELAY2.2, REEDRELAY3.2, REEDRELAY4.2, RELAY1.C1, RELAY2.C1, RELAY3.C1, RELAY4.C1, T3.S, T7.S, T9.S; no longer FB10.P$1, FB2.P$2, FB6.P$2, U$20.VCC, U$21.VCC, U$22.VCC, U$23.VCC, U$24.P$1, U$40.3, U$41.3, U$42.3, U$43.3
- net GND: now also C10.2, C11.2, C19.2, C9.1, FB5.P$1, REEDRELAY2.1, REEDRELAY3.1, T12.S, T13.S, T14.S, T15.S, T16.S, T17.S, T8.S, U$20.CS2, U$20.CS3, U$20.GND, U$21.CS2, U$21.CS3, U$21.GND, U$22.CS2, U$22.CS3, U$22.GND, U$23.CS2, U$23.CS3, U$23.GND, U$25.V-, U$29.V-; no longer FB9.P$1, T3.S, T4.S, T8.D, U$44.S
- net HV-: now also RELAY1.NO, RELAY1.P$5, RELAY2.NO, RELAY2.P$5, RELAY3.COM, RELAY3.NO, RELAY3.P$5, RELAY4.COM, RELAY4.NO, RELAY4.P$5
- net MEG-: now also JP3.1
- net N$103: now also FB2.P$2, T9.D; no longer FB5.P$1, U$44.D
- net N$114: now also FB6.P$2, T7.D; no longer FB2.P$1, T9.S
- net N$116: now also R46.1, T7.G, U$44.D; no longer ADC1.VDD, C10.1, C17.1, C9.2, IC1.+VS, R25.2, R26.2, R27.2, T9.D
- net N$117: now also ADC1.VDD, C10.1, C17.1, C19.1, C9.2, FB2.P$1, IC1.+VS, R25.2, R26.2, R27.2, U$25.V+; no longer C12.2, C13.1, C18.2, IC2.+VS, T11.D
- net N$118: now also U$25.IN-, U$25.OUT; no longer IC1.OUT
- net N$119: now also U$29.IN-, U$29.OUT; no longer IC2.OUT
- net N$26: now also R34.1, T3.G, T8.D; no longer U$20.CS2, U$20.CS3, U$20.GND, U$21.CS2, U$21.CS3, U$21.GND, U$22.CS2, U$22.CS3, U$22.GND, U$23.CS2, U$23.CS3, U$23.GND
- net N$49: now also RELAY1.COM, RELAY2.COM
- net N$5: no longer U2.EN
- net N$55: now also JP4.3, REEDRELAY1.4; no longer R34.2, T3.G
- net N$56: now also JP4.2, REEDRELAY2.4, REEDRELAY4.4; no longer T3.D, U$43.2
- net N$75: now also IC1.OUT, U$25.IN+; no longer ADC1.GND, C10.2, C9.1, FB1.P$2
- net N$80: now also JP4.1, REEDRELAY3.4; no longer R35.1, T4.G
- net N$89: now also REEDRELAY1.3, T5.D; no longer R37.1, T6.G
- net N$91: now also REEDRELAY4.3, T16.D; no longer T6.D, U$40.2
- net N$99: now also U$44.S
- net PMCM1: now also R36.1
- net PMCM2: now also R37.2
- net PMCM3: now also R60.1
- net PMCM4: now also R59.2
- net PRM2: now also R53.1
- net RCM1: now also R55.1; no longer R34.1
- net RCM2: now also R56.2; no longer R35.2
- net RCM3: now also R57.2; no longer R36.2
- net RCM4: now also R58.1; no longer R37.2
- net TO+BANANA: now also REEDRELAY1.1, REEDRELAY4.1
- net V1000: no longer U$42.4
- net V2500: no longer U$41.4
- net V500: no longer U$43.4
Other:
- note added: "5:27 - 500V 5:53 - 1000V 5:127 - 2500V 5:253 - 5000V"
- note added: "BANANA CONNECTER FOR HV MUST BE ADDED"
- note added: "NORMAL OPERATION PMCM1 and PMCM3 - ON PMCM2 and PMCM4 - OFF POSITIVE -GND OPERATION PMCM1 and PMCM4 - ON PMCM2 and PMCM3 - OFF NEGATIVE -GND OPERATION PMCM2 and PMCM4 - ON PMCM1 and PMCM3 - OFF"
- note added: "PULLUP TO ENABLE POWER SUPPLY"
- note added: "VOUTHV GOES TO MEG+ TER- MINAL"
- note removed: "12VA"
- note removed: "5:252 (VP/VS)"
- note removed: "NO CENTERTAP NEEDED IN THE SECONDARY SIDE"
- note removed: "TRANSFORMER RATIO 10: 504"
- moved on the sheet: ADC1, ADC2, ADC3, C1, C10, C12, C13, C14, C15, C16, C17, C18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

Commit message: Add I2C connection, Opamp for CS
Parts:
- removed R51: 10K, Ampparts:ERJ-2GEJ102X
- removed RELAY5: (no value), CAP_Diode_Megger:T9GS1L14-5
- removed U$24: 15uF, CAP_Diode_Megger:CAPACTORFORTRANSFORMER
- removed U$26, U$27: 100nF, powersupply:CC0402KRX5R7BB104
- removed U$3: 100nF, powersupply:CC0402KRX7R6BB104
- added C22, C32, C33: 100nF, powersupply:CC0402KRX5R7BB104
- added C29: 10uF, powersupply:CC1206ZKY5V7BB106
- added C34: 15uF, CAP_Diode_Megger:CAPACTORFORTRANSFORMER
- RDIS1: value 200M -> 100M
- renumbered SMD1 to CHV1, SMD10 to CHV6, SMD13 to CHV7, SMD14 to CHV8, SMD17 to CHV9, SMD18 to CHV10, SMD2 to CHV2, SMD21 to CHV11, SMD22 to CHV12, SMD25 to CHV13, SMD26 to CHV14, SMD29 to CHV15, SMD30 to CHV16, SMD33 to CHV17, SMD34 to CHV18, SMD37 to CHV19, SMD38 to CHV20, SMD5 to CHV33, SMD6 to CHV4, SMD9 to CHV5, U$1 to C20, U$10 to C27, U$12 to C28, U$16 to C30, U$17 to C31, U$2 to C21, U$4 to C23, U$5 to C24, U$6 to C25, U$7 to C26
Connections:
- net N$106 renamed VOLTAGEMODE
- net N$107 renamed CURRENTMODE
- net N$108 renamed MEGGERON
- net N$109 renamed VOLTGAGESELECTION
- net N$110 renamed ENTERFORMEGGER
- removed net N$112: S8.P, U$19.GEN/6GPIO25
- removed net N$113: R51.2, S8.S
- new net EMERGENCYSTOP: S8.S, U$19.GEN/6GPIO25
- net BATT+: now also C22.1; no longer U$3.1
- net GND: now also C22.2, C29.1, C32.2, C33.1, C34.P$2; no longer R51.1, U$24.P$2, U$26.1, U$27.2, U$3.2
- net N$111: now also S8.P
- net N$2: now also C32.1; no longer U$27.1
- net PIE5+: now also C29.2, C34.P$1; no longer U$24.P$1
- net TOATMEGAVCC: now also C33.2; no longer U$26.2
Other:
- moved on the sheet: ADC1, C10, C17, C19, C9, D1, DZ1, FB1, FB2, IC1, J1, J2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
